Commit message: commit before implementing reolute2 joints

File: src/mybot_description/urdf/mybot.xacro (robot description, xacro)
@@ -24,10 +24,10 @@
     <pose>0 0 0.0 0 0 0</pose>
     <inertial>
-      <mass value="15.0"/>
+      <mass value="100.0"/>
       <origin xyz="0.0 0 0.0" rpy=" 0 0 0"/>
       <inertia
-          ixx="0.1" ixy="0" ixz="0"
-          iyy="0.1" iyz="0"
-          izz="0.1"
+          ixx="8.4167" ixy="0" ixz="0"
+          iyy="40.417" iyz="0"
+          izz="48.667"
       />
     </inertial>
@@ -106,5 +106,5 @@
     <child link="axel_hinge_left"/>
     <limit effort="100" velocity="10" lower="-0.2" upper="0.2"/>
-    <safety_controller k_position="10" k_velocity="10" soft_lower_limit="-2" oft_upper_limitt="2"/>
+    <safety_controller k_position="10" k_velocity="10" soft_lower_limit="-2" soft_upper_limit="2"/>
     <joint_properties damping="0.1" friction="0.0"/>
   </joint>
@@ -137,10 +137,10 @@
     <child link="axel_hinge_right"/>
     <limit effort="100" velocity="10"  lower="-0.2" upper="0.2"/>
-    <safety_controller k_position="10" k_velocity="10" soft_lower_limit="-0.19" oft_upper_limitt="0.19"/>
+    <safety_controller k_position="10" k_velocity="10" soft_lower_limit="-0.19" soft_upper_limit="0.19"/>
     <joint_properties damping="0.0" friction="0.0"/>
   </joint>
   <link name="left_wheel_front">
     <collision name="collision">
-      <origin xyz="0.0 0 0.0" rpy="0 0 0"/>
+      <origin xyz="0.0 0 0.0" rpy="0 1.5707 1.5707"/>
       <geometry>
         <cylinder radius="0.08" length="0.05"/>
@@ -167,6 +167,6 @@
     <parent link="axel_hinge_left"/>
     <axis xyz="0 1 0" rpy="0 0 0"/>
-    <limit effort="100" velocity="100"/>
-    <joint_properties damping="1.0" friction="1.0"/>
+    <limit effort="1" velocity="0"/>
+    <joint_properties damping="10.0" friction="10.0"/>
   </joint>
   <link name="right_wheel_front">
@@ -197,10 +197,10 @@
     <parent link="axel_hinge_right"/>
     <axis xyz="0 1 0" rpy="0 0 0"/>
-    <limit effort="100" velocity="100"/>
-    <joint_properties damping="1.0" friction="1.0"/>
+    <limit effort="1" velocity="0"/>
+    <joint_properties damping="10.0" friction="10.0"/>
   </joint>
   <link name="left_wheel_back">
     <collision name="collision">
-      <origin xyz="0.0 0 0.0" rpy="0 0 0"/>
+      <origin xyz="0.0 0 0.0" rpy="0 1.5707 1.5707"/>
       <geometry>
         <cylinder radius="0.08" length="0.05"/>

Commit message: somehow working

File: src/mybot_description/urdf/mybot.xacro (robot description, xacro)
@@ -162,41 +162,37 @@
     </inertial>
   </link>
-  <joint type="continuous" name="left_wheel_front_hinge">
+  <joint name="left_wheel_front_hinge" type="fixed">
+    <axis xyz="0 1 0" rpy="0 0 0"/>
     <origin xyz="0.0 0.025 0.00" rpy="0 0 0"/>
+    <parent link="axel_hinge_left"/>
     <child link="left_wheel_front"/>
-    <parent link="axel_hinge_left"/>
+  </joint>
+  <link name="right_wheel_front">
+    <collision name="collision">
+      <origin xyz="0.0 0 0.0" rpy="0 1.5707 1.5707"/>
+      <geometry>
+        <cylinder radius="0.08" length="0.05"/>
+      </geometry>
+    </collision>
+    <visual name="right_wheel_front_visual">
+      <origin xyz="0.0 0 0.0" rpy="0 1.5707 1.5707"/>
+      <geometry>
+        <cylinder radius="0.08" length="0.05"/>
+      </geometry>
+    </visual>
+    <inertial>
+      <origin xyz="0.0 0 0.0" rpy="0 0 0"/>
+      <mass value="0.1"/>
+      <inertia
+        ixx=".1" ixy="0.0" ixz="0.0"
+        iyy=".1" iyz="0.0"
+        izz=".1"/>
+    </inertial>
+  </link>
+  <joint name="right_wheel_front_hinge" type="fixed">
     <axis xyz="0 1 0" rpy="0 0 0"/>
-    <limit effort="1" velocity="0"/>
-    <joint_properties damping="10.0" friction="10.0"/>
-  </joint>
-  <link name="right_wheel_front">
-    <collision name="collision">
-      <origin xyz="0.0 0 0.0" rpy="0 1.5707 1.5707"/>
-      <geometry>
-        <cylinder radius="0.08" length="0.05"/>
-      </geometry>
-    </collision>
-    <visual name="right_wheel_front_visual">
-      <origin xyz="0.0 0 0.0" rpy="0 1.5707 1.5707"/>
-      <geometry>
-        <cylinder radius="0.08" length="0.05"/>
-      </geometry>
-    </visual>
-    <inertial>
-      <origin xyz="0.0 0 0.0" rpy="0 0 0"/>
-      <mass value="0.1"/>
-      <inertia
-        ixx=".1" ixy="0.0" ixz="0.0"
-        iyy=".1" iyz="0.0"
-        izz=".1"/>
-    </inertial>
-  </link>
-  <joint type="continuous" name="right_wheel_front_hinge">
     <origin xyz="0.0 -0.025 0.00" rpy="0 0 0"/>
+    <parent link="axel_hinge_right"/>
     <child link="right_wheel_front"/>
-    <parent link="axel_hinge_right"/>
-    <axis xyz="0 1 0" rpy="0 0 0"/>
-    <limit effort="1" velocity="0"/>
-    <joint_properties damping="10.0" friction="10.0"/>
   </joint>
   <link name="left_wheel_back">
@@ -214,6 +210,6 @@
     </visual>
     <inertial>
-      <origin xyz="0.0 0 -0.0" rpy="0 0 0"/>
-      <mass value="0.01"/>
+      <origin xyz="0.0 0 -0.0" rpy="0 1.5707 1.5707"/>
+      <mass value="0.1"/>
       <inertia
         ixx=".1" ixy="0.0" ixz="0.0"
@@ -223,5 +219,5 @@
   </link>
   <joint type="continuous" name="left_wheel_back_joint">
-    <origin xyz="-0.12 0.15 -0.03" rpy="0 0 0"/>
+    <origin xyz="-0.15 0.15 -0.03" rpy="0 0 0"/>
     <child link="left_wheel_back"/>
     <parent link="base_link"/>
@@ -243,6 +239,6 @@
     </visual>
     <inertial>
-      <origin xyz="0.0 0 0.0" rpy="0 0 0"/>
-      <mass value="0.01"/>
+      <origin xyz="0.0 0 0.0" rpy="0 1.5707 1.5707"/>
+      <mass value="0.1"/>
       <inertia
         ixx=".1" ixy="0.0" ixz="0.0"
@@ -252,5 +248,5 @@
   </link>
   <joint type="continuous" name="right_wheel_back_joint">
-    <origin xyz="-0.12 -0.15 -0.03" rpy="0 0 0"/>
+    <origin xyz="-0.15 -0.15 -0.03" rpy="0 0 0"/>
     <child link="right_wheel_back"/>
     <parent link="base_link"/>

Commit message: finaly a working rc car with ackerman steering model, still front wheels are not aligned with axis

File: src/mybot_description/urdf/mybot.xacro (robot description, xacro)
@@ -196,4 +196,33 @@
     <child link="right_wheel_front"/>
   </joint>
+ <link name="back_axel">
+    <collision name="collision">
+      <origin xyz="0.0 0 0.0" rpy="0 1.5707 1.5707"/>
+      <geometry>
+        <cylinder radius="0.007" length="0.25"/>
+      </geometry>
+    </collision>
+    <visual name="axel_visual">
+      <origin xyz="0.0 0.0 0.0" rpy="0 1.5707 1.5707"/>
+      <geometry>
+        <cylinder radius="0.007" length="0.25"/>
+      </geometry>
+    </visual>
+    <inertial>
+      <origin xyz="0.0 0 0.0" rpy="0 0 0"/>
+      <mass value="5"/>
+      <inertia
+        ixx=".1" ixy="0.0" ixz="0.0"
+        iyy=".1" iyz="0.0"
+        izz=".1"/>
+    </inertial>
+  </link>
+  <joint type="continuous" name="back_axel_joint">
+    <origin xyz="-0.15 0.0 -0.03" rpy="0 0 0"/>
+    <child link="back_axel"/>
+    <parent link="base_link"/>
+    <axis xyz="0 1 0" rpy="0 0 0"/>
+    <dynamics damping = "0.7" />
+  </joint>
   <link name="left_wheel_back">
     <collision name="collision">
@@ -218,10 +247,9 @@
     </inertial>
   </link>
-  <joint type="continuous" name="left_wheel_back_joint">
-    <origin xyz="-0.15 0.15 -0.03" rpy="0 0 0"/>
+  <joint type="fixed" name="left_wheel_back_joint">
+    <origin xyz="0 0.15 0" rpy="0 0 0"/>
     <child link="left_wheel_back"/>
-    <parent link="base_link"/>
-    <axis xyz="0 1 0" rpy="0 0 0"/>
-    <dynamics damping = "0.7" />
+    <parent link="back_axel"/>
+    <axis xyz="0 1 0" rpy="0 0 0"/>
   </joint>
   <link name="right_wheel_back">
@@ -247,10 +275,9 @@
     </inertial>
   </link>
-  <joint type="continuous" name="right_wheel_back_joint">
-    <origin xyz="-0.15 -0.15 -0.03" rpy="0 0 0"/>
+  <joint type="fixed" name="right_wheel_back_joint">
+    <origin xyz="0 -0.15 0" rpy="0 0 0"/>
     <child link="right_wheel_back"/>
-    <parent link="base_link"/>
-    <axis xyz="0 1 0" rpy="0 0 0"/>
-    <dynamics damping = "0.7" />
+    <parent link="back_axel"/>
+    <axis xyz="0 1 0" rpy="0 0 0"/>
   </joint>
   <link name="camera">
@@ -309,5 +336,5 @@
   <transmission name="tran1">
     <type>transmission_interface/SimpleTransmission</type>
-    <joint name="left_wheel_back_joint">
+    <joint name="back_axel_joint">
       <hardwareInterface>hardware_interface/EffortJointInterface</hardwareInterface>
     </joint>
@@ -319,5 +346,5 @@
   <transmission name="tran2">
     <type>transmission_interface/SimpleTransmission</type>
-    <joint name="right_wheel_back_joint">
+    <joint name="axel_hinge_right_joint">
       <hardwareInterface>hardware_interface/EffortJointInterface</hardwareInterface>
     </joint>
@@ -329,18 +356,8 @@
   <transmission name="tran3">
     <type>transmission_interface/SimpleTransmission</type>
-    <joint name="axel_hinge_right_joint">
+    <joint name="axel_hinge_left_joint">
       <hardwareInterface>hardware_interface/EffortJointInterface</hardwareInterface>
     </joint>
     <actuator name="motor3">
-      <hardwareInterface>hardware_interface/EffortJointInterface</hardwareInterface>
-      <mechanicalReduction>1</mechanicalReduction>
-    </actuator>
-  </transmission>
-  <transmission name="tran4">
-    <type>transmission_interface/SimpleTransmission</type>
-    <joint name="axel_hinge_left_joint">
-      <hardwareInterface>hardware_interface/EffortJointInterface</hardwareInterface>
-    </joint>
-    <actuator name="motor4">
       <hardwareInterface>hardware_interface/EffortJointInterface</hardwareInterface>
       <mechanicalReduction>1</mechanicalReduction>

Commit message: size adjusted

File: src/mybot_description/urdf/mybot.xacro (robot description, xacro)
@@ -33,5 +33,5 @@
       <origin xyz="0.0 0 0.0" rpy="0 1.5707 1.5707"/>
       <geometry>
-        <cylinder radius="0.007" length="0.25"/>
+        <cylinder radius="0.005" length="0.20"/>
       </geometry>
     </collision>
@@ -39,5 +39,5 @@
       <origin xyz="0.0 0.0 0.0" rpy="0 1.5707 1.5707"/>
       <geometry>
-        <cylinder radius="0.007" length="0.25"/>
+        <cylinder radius="0.005" length="0.20"/>
       </geometry>
     </visual>
@@ -48,4 +48,5 @@
     <parent link="chassis"/>
     <axis xyz="0 1 0" rpy="0 0 0"/>
+    <limit effort="10" velocity="100" />
   </joint>
   <!-- Add the left rear wheel with its joints and tranmissions -->
