Commit message: back axel added but not connected and size has to be adjusted

File: src/mybot_description/urdf/macros.xacro (robot description, xacro)
@@ -8,4 +8,11 @@
                           iyy="0.050409"   iyz="0"
                                            izz="0.05865" />
+</xacro:macro>
+<xacro:macro name="back_axel_inertial_params">
+  <origin xyz="0 0 -0.0225" rpy="0 0 0" />
+  <mass value="0.34055" />
+  <inertia ixx="0.00026046" ixy="0"          ixz="0"
+                            iyy="0.00026046" iyz="0"
+                                             izz="0.00041226" />
 </xacro:macro>
 <xacro:macro name="left_wheels_inertial_params">

File: src/mybot_description/urdf/mybot.xacro (robot description, xacro)
@@ -25,4 +25,28 @@
     <child link="chassis_inertia" />
   </joint>
+  <!-- Add the rear axel with its joints and transmissions    -->
+  <link name="back_axel">
+    <inertial>
+      <xacro:left_wheels_inertial_params />
+    </inertial>
+    <collision name="collision">
+      <origin xyz="0.0 0 0.0" rpy="0 1.5707 1.5707"/>
+      <geometry>
+        <cylinder radius="0.007" length="0.25"/>
+      </geometry>
+    </collision>
+    <visual name="axel_visual">
+      <origin xyz="0.0 0.0 0.0" rpy="0 1.5707 1.5707"/>
+      <geometry>
+        <cylinder radius="0.007" length="0.25"/>
+      </geometry>
+    </visual>
+      </link>
+  <joint type="continuous" name="back_axel_joint">
+    <origin xyz="0.0 0.0 0.0" rpy="0 0 0"/>
+    <child link="back_axel"/>
+    <parent link="chassis"/>
+    <axis xyz="0 1 0" rpy="0 0 0"/>
+  </joint>
   <!-- Add the left rear wheel with its joints and tranmissions -->
   <link name="left_rear_wheel">

Commit message: got fed up again with this shitting gazebo ... gonna revert back to the mit version to try and get that working completely

File: src/mybot_description/urdf/macros.xacro (robot description, xacro)
@@ -104,8 +104,8 @@
     <type>transmission_interface/SimpleTransmission</type>
     <joint name="${name}_joint">
-      <hardwareInterface>EffortJointInterface</hardwareInterface>
+      <hardwareInterface>hardware_interface/EffortJointInterface</hardwareInterface>
     </joint>
     <actuator name="${name}_motor">
-      <hardwareInterface>EffortJointInterface</hardwareInterface>
+      <hardwareInterface>hardware_interface/EffortJointInterface</hardwareInterface>
       <mechanicalReduction>1</mechanicalReduction>
     </actuator>
@@ -116,8 +116,8 @@
     <type>transmission_interface/SimpleTransmission</type>
     <joint name="${name}_joint">
-      <hardwareInterface>EffortJointInterface</hardwareInterface>
+       <hardwareInterface>hardware_interface/EffortJointInterface</hardwareInterface>
     </joint>
     <actuator name="${name}_motor">
-      <hardwareInterface>EffortJointInterface</hardwareInterface>
+      <hardwareInterface>hardware_interface/EffortJointInterface</hardwareInterface>
       <mechanicalReduction>1</mechanicalReduction>
     </actuator>

File: src/mybot_description/urdf/mybot.xacro (robot description, xacro)
@@ -26,5 +26,5 @@
   </joint>
   <!-- Add the rear axel with its joints and transmissions    -->
-  <link name="back_axel">
+  <link name="rear_axel">
     <inertial>
       <xacro:left_wheels_inertial_params />
@@ -36,5 +36,5 @@
       </geometry>
     </collision>
-    <visual name="axel_visual">
+    <visual name="rear_axel_visual">
       <origin xyz="0.0 0.0 0.0" rpy="0 1.5707 1.5707"/>
       <geometry>
@@ -43,12 +43,13 @@
     </visual>
       </link>
-  <joint type="continuous" name="back_axel_joint">
+  <joint type="continuous" name="rear_axel_joint">
     <origin xyz="0.0 0.0 0.0" rpy="0 0 0"/>
-    <child link="back_axel"/>
+    <child link="rear_axel"/>
     <parent link="chassis"/>
     <axis xyz="0 1 0" rpy="0 0 0"/>
     <limit effort="10" velocity="100" />
   </joint>
-  <!-- Add the left rear wheel with its joints and tranmissions -->
+  <xacro:wheel_transmission name="rear_axel" />
+  <!-- Add the left rear wheel with its joints -->
   <link name="left_rear_wheel">
     <inertial>
@@ -59,17 +60,14 @@
       <material name="black" />
     </visual>
-    <collision>robot
+    <collision>
       <xacro:left_wheels_collision_geometry />
     </collision>
   </link>
-  <joint name="left_rear_wheel_joint" type="continuous">
+  <joint name="left_rear_wheel_joint" type="fixed">
     <origin xyz="0 0.1 0" rpy="1.5708 0 0" />
-    <parent link="chassis" />
+    <parent link="rear_axel" />
     <child link="left_rear_wheel" />
-    <axis xyz="0 0 -1" />
-    <limit effort="10" velocity="100" />
-  </joint>
-  <xacro:wheel_transmission name="left_rear_wheel" />
-  <!-- Add the right rear wheel with its joints and tranmissions -->
+  </joint>
+  <!-- Add the right rear wheel with its joints -->
   <link name="right_rear_wheel">
     <inertial>
@@ -84,12 +82,9 @@
     </collision>
   </link>
-  <joint name="right_rear_wheel_joint" type="continuous">
+  <joint name="right_rear_wheel_joint" type="fixed">
     <origin xyz="0 -0.1 0" rpy="1.5708 0 0" />
-    <parent link="chassis" />
+    <parent link="rear_axel" />
     <child link="right_rear_wheel" />
-    <axis xyz="0 0 -1" />
-    <limit effort="10" velocity="100" />
-  </joint>
-  <xacro:wheel_transmission name="right_rear_wheel" />
+  </joint>
   <!-- Add the left steering hinge with its joints and tranmissions -->
   <link name="left_steering_hinge">
@@ -111,5 +106,5 @@
   <xacro:steering_hinge_transmission name="left_steering_hinge" />
   <!-- Add the right steering hinge with its joints and tranmissions -->
-  <link name="right_steering_hinge">
+  <!--link name="right_steering_hinge">
     <inertial>
       <xacro:steering_hinge_inertial_params />
@@ -120,5 +115,5 @@
     </visual>
   </link>
-  <joint name="right_steering_hinge_joint" type="continuous">
+  <joint name="right_steering_hinge_joint" type="revolute">
     <origin xyz="0.325 -0.1 0" rpy="0 1.5708 0" />
     <parent link="chassis" />
@@ -127,5 +122,5 @@
     <limit lower="-1.0" upper="1.0" effort="10" velocity="100" />
   </joint>
-  <xacro:steering_hinge_transmission name="right_steering_hinge" />
+  <xacro:steering_hinge_transmission name="right_steering_hinge" /-->
   <!-- Add the left front wheel with its joints and tranmissions -->
   <link name="left_front_wheel">
@@ -141,14 +136,12 @@
     </collision>
   </link>
-  <joint name="left_front_wheel_joint" type="continuous">
+  <joint name="left_front_wheel_joint" type="fixed">
     <origin xyz="0 0 0" rpy="1.5708 0 0" />
     <parent link="left_steering_hinge" />
     <child link="left_front_wheel" />
     <axis xyz="0 0 -1" />
-    <limit effort="10" velocity="100" />
-  </joint>
-  <xacro:wheel_transmission name="left_front_wheel" />
+  </joint>
   <!-- Add the left front wheel with its joints and tranmissions -->
-  <link name="right_front_wheel">
+  <!--link name="right_front_wheel">
     <inertial>
       <xacro:right_wheels_inertial_params />
@@ -169,5 +162,5 @@
     <limit effort="10" velocity="100"/>
   </joint>
-  <xacro:wheel_transmission name="right_front_wheel" />
+  <xacro:wheel_transmission name="right_front_wheel" /-->
   <!-- Add Hokuyo laser scanner -->
   <link name="laser">

Commit message: finaly figured out a way that could be working! effort controller instead of velocity controller needs higher resistance values to stop continuous movement and a self written pid controller for speed control

File: src/mybot_description/urdf/macros.xacro (robot description, xacro)
@@ -97,8 +97,8 @@
     <type>transmission_interface/SimpleTransmission</type>
     <joint name="${name}_joint">
-      <hardwareInterface>EffortJointInterface</hardwareInterface>
+      <hardwareInterface>hardware_interface/EffortJointInterface</hardwareInterface>
     </joint>
     <actuator name="${name}_motor">
-      <hardwareInterface>EffortJointInterface</hardwareInterface>
+      <hardwareInterface>hardware_interface/EffortJointInterface</hardwareInterface>
       <mechanicalReduction>1</mechanicalReduction>
     </actuator>
@@ -109,8 +109,8 @@
     <type>transmission_interface/SimpleTransmission</type>
     <joint name="${name}_joint">
-      <hardwareInterface>EffortJointInterface</hardwareInterface>
+      <hardwareInterface>hardware_interface/EffortJointInterface</hardwareInterface>
     </joint>
     <actuator name="${name}_motor">
-      <hardwareInterface>EffortJointInterface</hardwareInterface>
+      <hardwareInterface>hardware_interface/EffortJointInterface</hardwareInterface>
       <mechanicalReduction>1</mechanicalReduction>
     </actuator>

File: src/mybot_description/urdf/mybot.xacro (robot description, xacro)
@@ -82,5 +82,5 @@
     <child link="left_steering_hinge" />
     <axis xyz="-1 0 0" />
-    <limit lower="-1.0" upper="1.0" effort="10" velocity="100" />
+    <limit lower="-0.5" upper="0.5" effort="1" velocity="1" />
   </joint>
   <xacro:steering_hinge_transmission name="left_steering_hinge" />
@@ -95,10 +95,10 @@
     </visual>
   </link>
-  <joint name="right_steering_hinge_joint" type="continuous">
+  <joint name="right_steering_hinge_joint" type="revolute">
     <origin xyz="0.325 -0.1 0" rpy="0 1.5708 0" />
     <parent link="chassis" />
     <child link="right_steering_hinge" />
     <axis xyz="-1 0 0" />
-    <limit lower="-1.0" upper="1.0" effort="10" velocity="100" />
+    <limit lower="-0.5" upper="0.5" effort="1" velocity="1" />
   </joint>
   <xacro:steering_hinge_transmission name="right_steering_hinge" />
